File: ModdedCard/RolandMpuImcMod.sch (KiCad schematic (older format))
At the start: 123 parts, among them IC1 LC3517, IC10 74LS138, IC11 74LS573, IC12 74LS86_P, IC13 74LS688, IC14 HEF4093B, IC15 74LS688, IC16 5218, IC17 H11L1, IC2 HG62E08, IC3 HD6801VD855P, IC4 74LS05, IC5 74LS02, IC6 74LS05, IC7 74LS32, IC8 74LS04, IC9 74LS74, J1 DB9_Female_MountingHoles, J2 BUS_MCA, J3 Conn_01x01, J4 Conn_01x01, J5 Conn_01x01, J6 Conn_01x01, Q1 2SC1815, Q2 2SC1815, Q3 2SC1815, Q4 2SC1815, Q5 2SC1815, X1 Crystal

Commit message: Fix IC3 pin swap and a few part numbers
Parts:
- C1, C10, C11, C12, C13, C14, C15, C17, C18, C19, C20, C21, C22, C24, C25, C26, C27, C28, C29, C3, C30, C31, C32, C34, C35, C4, C5A1, C5B1, C6, C7, C8, C9: symbol C_Small -> Device:C_Small
- C16, C2, C23, C33: symbol CP1_Small -> Device:CP1_Small
- D1, D2, D3: symbol D_Small_ALT -> Device:D_Small_ALT
- FL1, FL2, FL3, FL4, FL5, FL6, FL7, FL8, FL9: symbol EMI_Filter_C -> Device:EMI_Filter_C
- IC1: value LC3517 -> LC3517 (or HY6116AP-10); symbol LC3517 -> Roland:LC3517
- IC10: symbol 74LS138 -> RolandMpuImcMod-rescue:74LS138
- IC11: value 74LS573 -> 74ALS573; symbol 74LS573 -> RolandMpuImcMod-rescue:74LS573; Mouser (none) -> 595-SN74ALS573CN
- IC12: symbol 74LS86_P -> Roland:74LS86_P
- IC13, IC15: symbol 74LS688 -> RolandMpuImcMod-rescue:74LS688
- IC14: symbol HEF4093B -> RolandMpuImcMod-rescue:HEF4093B
- IC16: symbol LM2904 -> RolandMpuImcMod-rescue:LM2904
- IC17: symbol H11L1 -> RolandMpuImcMod-rescue:H11L1
- IC2: symbol HG62E08 -> Roland:HG62E08
- IC3: symbol HD6801VD855P -> Roland:HD6801VD855P
- IC4, IC6: symbol 74LS05 -> RolandMpuImcMod-rescue:74LS05
- IC5: symbol 74LS02 -> RolandMpuImcMod-rescue:74LS02
- IC7: symbol 74LS32 -> RolandMpuImcMod-rescue:74LS32
- IC8: symbol 74LS04 -> RolandMpuImcMod-rescue:74LS04
- IC9: symbol 74LS74 -> RolandMpuImcMod-rescue:74LS74
- IRQ1: symbol Conn_02x06_Odd_Even -> RolandMpuImcMod-rescue:Conn_02x06_Odd_Even
- J1: symbol DB9_Female_MountingHoles -> RolandMpuImcMod-rescue:DB9_Female_MountingHoles; Mouser 806-K22X-E9S-NJ -> 571-2311765-1
- J2: symbol BUS_MCA -> Roland:BUS_MCA
- J3, J4, J5, J6: symbol Conn_01x01 -> RolandMpuImcMod-rescue:Conn_01x01
- L2: symbol L_Core_Ferrite_Small -> Device:L_Core_Ferrite_Small
- Q1, Q2, Q3, Q4, Q5: symbol 2SC1815 -> RolandMpuImcMod-rescue:2SC1815
- R1, R10, R11, R12, R13, R14, R15, R16, R17, R19, R2, R21, R22, R23, R24, R25, R26, R27, R28, R29, R3, R30, R31, R32, R33, R34, R35, R36, R37, R38, R39, R4, R40, R41, R43, R44, R5, R6, R7, R8, R9: symbol R_Small -> Device:R_Small
- R18, R20: symbol R_Small -> Device:R_Small; Mouser 603-CFR-12JB-52-150R -> 603-CFR-12JB-52-180R
- RA1: symbol R_Network08 -> Device:R_Network08
- X1: symbol Crystal -> Device:Crystal
Connections:
- net IRQ9: no longer IC6.6, IRQ1.10 (Pin_10), IRQ1.12 (Pin_12), IRQ1.2 (Pin_2), IRQ1.4 (Pin_4), IRQ1.6 (Pin_6), IRQ1.8 (Pin_8)
- net VCCF: now reaches C14.1, C19.1, IC12.14 (VCC), IC12.5 (IN2), IC14.14 (VCC), L2.1
- net VCCF: now also IC12.14 (VCC), IC12.14 (VCC), IC12.14 (VCC)
- net at IC2.16 (NCS2): now also IC3.26 (P43); no longer IC3.25 (P43)
- new net: IC6.6, IRQ1.10 (Pin_10), IRQ1.12 (Pin_12), IRQ1.2 (Pin_2), IRQ1.4 (Pin_4), IRQ1.6 (Pin_6), IRQ1.8 (Pin_8)
Other:
- note added: "IRQ9 is Roland's default\nbut may conflict with\nSCSI on certain PS/2s."
